Commit message: A lot Changed Iris.xacro added camera Added robot state and joint state publishers Added perception and msgs modules The perception module has the camera library and obstacle detectors Tuned the vision to recognize red and green obstacles 2D to 3D projection is mostly good but can be tuned with knowledge of obstacle bounding boxes

File: external/rotors_description/urdf/iris.xacro (robot description, xacro)
@@ -130,3 +130,70 @@
     <xacro:insert_block name="rotor_inertia" />
   </xacro:vertical_rotor>
+  <xacro:property name="JOINT_KP" value="1e15"/>
+  <xacro:property name="JOINT_KD" value="1e13"/>
+  <xacro:property name="JOINT_MU1" value="0.2"/>
+  <xacro:property name="JOINT_MU2" value="0.2"/>
+  <xacro:property name="JOINT_FRICTION" value="0.1"/>
+  <xacro:property name="JOINT_DAMPING" value="0.01"/>
+  <link name="${namespace}/camera" >
+            <inertial>
+                <mass value="0.01"/>
+                <origin rpy="0  0  0" xyz="0 0 0"/>
+                <inertia ixx="1e-9" ixy="0" ixz="0"
+                         iyy="1e-9" iyz="0"
+                         izz="1e-9"/>
+            </inertial>
+        </link>
+        <joint name="${namespace}/camera" type="fixed">
+            <parent link="${namespace}/base_link"/>
+            <child link="${namespace}/camera"/>
+            <origin rpy="0 0 0" xyz="0.015 0.00145 0.04740"/>
+            <axis xyz="0  0  0"/>
+            <dynamics damping="${JOINT_DAMPING}" friction="${JOINT_FRICTION}" />
+            <limit effort="0" lower="0" upper="0" velocity="0"/>
+        </joint>
+        <gazebo reference="${namespace}/camera">
+            <sensor type="camera" name="main_camera" >
+                <always_on>1</always_on>
+                <visualize>1</visualize>
+                <update_rate>30</update_rate>
+                <camera>
+                    <horizontal_fov>1.047</horizontal_fov>
+                    <image>
+                        <width>320</width>
+                        <height>240</height>
+                        <format>R8G8B8</format>
+                    </image>
+                    <clip>
+                        <near>0.1</near>
+                        <far>100</far>
+                    </clip>
+                    <noise>
+                        <type>gaussian</type>
+                        <mean>0</mean>
+                        <stddev>0.007</stddev>
+                    </noise>
+                </camera>
+<!--                <plugin  filename='libgazebo_ros_camera.so' name='camera_controller'>-->
+<!--                    <alwaysOn>true</alwaysOn>-->
+<!--                    <updateRate>0.0</updateRate>-->
+<!--                    <cameraName>camera</cameraName>-->
+<!--                    <imageTopicName>image_raw</imageTopicName>-->
+<!--                    <cameraInfoTopicName>camera_info</cameraInfoTopicName>-->
+<!--                    <frameName>camera_link</frameName>-->
+<!--                    <hackBaseline>0.07</hackBaseline>-->
+<!--                    <distortionK1>0.0</distortionK1>-->
+<!--                    <distortionK2>0.0</distortionK2>-->
+<!--                    <distortionK3>0.0</distortionK3>-->
+<!--                    <distortionT1>0.0</distortionT1>-->
+<!--                    <distortionT2>0.0</distortionT2>-->
+<!--                </plugin>-->
+            </sensor>
+        </gazebo>
+        <gazebo reference="${namespace}/camera">
+            <kp>${JOINT_KP}</kp>
+            <kd>${JOINT_KD}</kd>
+            <mu1>${JOINT_MU1}</mu1>
+            <mu2>${JOINT_MU2}</mu2>
+        </gazebo>
 </robot>
